File: pcb/original/Madromys-orig.kicad_pcb (KiCad board)
At the start: 4 copper layers, 62 x 68 mm, 83 parts

Commit message: pcb: add holes for an extra button on GP12
Add two plated holes (GP12 and GND, 2.54 mm pitch) above LED.D.1.
GP12 is the former LED data line, which is free because the LEDs are
not mounted. Update the board files, Gerbers, previews and READMEs of
both variants.

Co-Authored-By: Claude Opus 5.5 <noreply@anthropic.com>
Claude-Session: https://claude.ai/code/session_018VxjY8mbESBV2UQ3jTsC2n
Parts:
- added BTN.J.9: EXT BUTTON, EXT_BUTTON_2x1, F.Cu at (170.0, 93.4)
Routing:
- net LEDData: track 24.6 -> 28.9 mm
Other:
- board text added: "GND"
- board text added: "GP12"
